File: Schematic-PCB/motordriver/motordriver-001-20250215/motordriver-001-20250215.kicad_sch (KiCad schematic)
At the start: 0 parts

Commit message: Update MD回路駆動部分完成
信号入力部分・ロジック電源供給部分はまだ
Parts:
- added C1, C2: 4.7u, symbol Device:C_Small
- added C10, C12, C6, C8: 220n, symbol Device:C_Small
- added C11, C5, C7, C9: 22n, symbol Device:C_Small
- added C3, C4: 0.1u, symbol Device:C_Small
- added J1: VIN, symbol Connector:Conn_01x02_Pin
- added J2: MOTOR-1, symbol Connector:Conn_01x02_Pin
- added J3: MOTOR-2, symbol Connector:Conn_01x02_Pin
- added J4: MOTOR-3, symbol Connector:Conn_01x02_Pin
- added J5: MOTOR-4, symbol Connector:Conn_01x02_Pin
- added R1, R13, R5, R9: 10K, symbol Device:R_Small
- added R10, R14, R2, R6: NP, symbol Device:R_Small
- added R11, R15, R3, R7: 20K, symbol Device:R_Small
- added R12, R16, R4, R8: 2.49K, symbol Device:R_Small
- added U1, U2, U3, U4: ~, symbol 2025-motordriver:DRV8874
Connections:
- new net: C12.1, U4.12 (VCP)
- new net: C11.2, U4.13 (CPH)
- new net: C11.1, U4.14 (CPL)
- new net: R16.1, U4.6 (IPROPI)
- new net: C8.1, U2.12 (VCP)
- new net: R8.1, U2.6 (IPROPI)
- new net: C5.1, U1.14 (CPL)
- new net: C5.2, U1.13 (CPH)
- new net: C6.1, U1.12 (VCP)
- new net: C7.2, U2.13 (CPH)
- new net: C7.1, U2.14 (CPL)
- new net: R12.1, U3.6 (IPROPI)
- new net: C9.1, U3.14 (CPL)
- new net: C9.2, U3.13 (CPH)
- new net: R4.1, U1.6 (IPROPI)
- new net: C10.1, U3.12 (VCP)
- new net +3.3V: R1.1, R13.1, R5.1, R9.1, U1.3 (nSLEEP), U2.3 (nSLEEP), U3.3 (nSLEEP), U4.3 (nSLEEP)
- new net EN-1: U1.1 (EN/IN1)
- new net EN-2: U2.1 (EN/IN1)
- new net EN-3: U3.1 (EN/IN1)
- new net EN-4: U4.1 (EN/IN1)
- new net GND: C1.2, C2.2, C3.2, C4.2, J1.2 (Pin_2), R10.2, R11.2, R12.2, R14.2, R15.2, R16.2, R2.2, R3.2, R4.2, R6.2, R7.2, R8.2, U1.15 (GND), U1.16 (PMODE), U1.17 (GND), U1.9 (PGND), U2.15 (GND), U2.16 (PMODE), U2.17 (GND), U2.9 (PGND), U3.15 (GND), U3.16 (PMODE), U3.17 (GND), U3.9 (PGND), U4.15 (GND), U4.16 (PMODE), U4.17 (GND), U4.9 (PGND)
- new net IMODE-1: R3.1, U1.7 (IMODE)
- new net IMODE-2: R7.1, U2.7 (IMODE)
- new net IMODE-3: R11.1, U3.7 (IMODE)
- new net IMODE-4: R15.1, U4.7 (IMODE)
- new net OUT1-1: J2.1 (Pin_1), U1.8 (OUT1)
- new net OUT1-2: J3.1 (Pin_1), U2.8 (OUT1)
- new net OUT1-3: J4.1 (Pin_1), U3.8 (OUT1)
- new net OUT1-4: J5.1 (Pin_1), U4.8 (OUT1)
- new net OUT2-1: J2.2 (Pin_2), U1.10 (OUT2)
- new net OUT2-2: J3.2 (Pin_2), U2.10 (OUT2)
- new net OUT2-3: J4.2 (Pin_2), U3.10 (OUT2)
- new net OUT2-4: J5.2 (Pin_2), U4.10 (OUT2)
- new net PH-1: U1.2 (PH/IN2)
- new net PH-2: U2.2 (PH/IN2)
- new net PH-3: U3.2 (PH/IN2)
- new net PH-4: U4.2 (PH/IN2)
- new net VCC: C1.1, C10.2, C12.2, C2.1, C3.1, C4.1, C6.2, C8.2, J1.1 (Pin_1), U1.11 (VM), U2.11 (VM), U3.11 (VM), U4.11 (VM)
- new net VREF-1: R1.2, R2.1, U1.5 (VREF)
- new net VREF-2: R5.2, R6.1, U2.5 (VREF)
- new net VREF-3: R10.1, R9.2, U3.5 (VREF)
- new net VREF-4: R13.2, R14.1, U4.5 (VREF)
- no-connect marks 0 -> 4
Other:
- note added: "MOTOR-1"
- note added: "MOTOR-2"
- note added: "MOTOR-3"
- note added: "MOTOR-4"
- note added: "OUTPUT"
- note added: "VIN"
