File: Schematic-PCB/line/line-001-20240304/line-001-20240304.kicad_sch (KiCad schematic)
At the start: 0 parts

Commit message: update: センサ部分を作った
Parts:
- added J1: Conn_01x03_Pin, symbol Connector:Conn_01x03_Pin
- added R1, R10, R11, R12, R13, R14, R15, R16, R17, R18, R19, R2, R20, R21, R22, R23, R24, R25, R26, R27, R28, R29, R3, R30, R4, R5, R6, R7, R8, R9: R, symbol Device:R
- added U1, U10, U11, U12, U13, U14, U15, U16, U17, U18, U19, U2, U20, U21, U22, U23, U24, U25, U26, U27, U28, U29, U3, U30, U4, U5, U6, U7, U8, U9: ~, symbol @2025-line:B19H1LS
Connections:
- net +5V: now also J1.1 (Pin_1), U1.1 (+), U10.1 (+), U11.1 (+), U12.1 (+), U13.1 (+), U14.1 (+), U15.1 (+), U16.1 (+), U17.1 (+), U18.1 (+), U19.1 (+), U2.1 (+), U20.1 (+), U21.1 (+), U22.1 (+), U23.1 (+), U24.1 (+), U25.1 (+), U26.1 (+), U27.1 (+), U28.1 (+), U29.1 (+), U3.1 (+), U30.1 (+), U4.1 (+), U5.1 (+), U6.1 (+), U7.1 (+), U8.1 (+), U9.1 (+)
- new net +3.3V: J1.2 (Pin_2)
- new net GND: J1.3 (Pin_3), R1.2, R10.2, R11.2, R12.2, R13.2, R14.2, R15.2, R16.2, R17.2, R18.2, R19.2, R2.2, R20.2, R21.2, R22.2, R23.2, R24.2, R25.2, R26.2, R27.2, R28.2, R29.2, R3.2, R30.2, R4.2, R5.2, R6.2, R7.2, R8.2, R9.2
- new net line-00: R1.1, U1.2 (-)
- new net line-01: R2.1, U2.2 (-)
- new net line-02: R3.1, U3.2 (-)
- new net line-03: R4.1, U4.2 (-)
- new net line-04: R5.1, U5.2 (-)
- new net line-05: R6.1, U6.2 (-)
- new net line-06: R7.1, U7.2 (-)
- new net line-07: R8.1, U8.2 (-)
- new net line-08: R9.1, U9.2 (-)
- new net line-09: R10.1, U10.2 (-)
- new net line-10: R11.1, U11.2 (-)
- new net line-11: R12.1, U12.2 (-)
- new net line-12: R13.1, U13.2 (-)
- new net line-13: R14.1, U14.2 (-)
- new net line-14: R15.1, U15.2 (-)
- new net line-15: R16.1, U16.2 (-)
- new net line-16: R17.1, U17.2 (-)
- new net line-17: R18.1, U18.2 (-)
- new net line-18: R19.1, U19.2 (-)
- new net line-19: R20.1, U20.2 (-)
- new net line-20: R21.1, U21.2 (-)
- new net line-21: R22.1, U22.2 (-)
- new net line-22: R23.1, U23.2 (-)
- new net line-23: R24.1, U24.2 (-)
- new net line-24: R25.1, U25.2 (-)
- new net line-25: R26.1, U26.2 (-)
- new net line-26: R27.1, U27.2 (-)
- new net line-27: R28.1, U28.2 (-)
- new net line-28: R29.1, U29.2 (-)
- new net line-29: R30.1, U30.2 (-)

Commit message: Summary (required)
Parts:
- added U31: ATMEGA2560-16AU, ATMEGA2560-16AU:QFP50P1600X1600X120-100N, symbol ATMEGA2560-16AU:ATMEGA2560-16AU
Connections:
- net +5V: now also U31.10 (VCC), U31.31 (VCC), U31.61 (VCC), U31.80 (VCC)
- net GND: now also U31.11 (GND), U31.32 (GND), U31.62 (GND), U31.81 (GND), U31.99 (GND)
